Commit message: Made changes

File: eddiebot_description/urdf/stacks/base.urdf.xacro (robot description, xacro)
@@ -220,5 +220,5 @@
       <axis xyz="0 1 0"/>
     </joint>
-    <ros2_control name="GazeboSimSystem" type="system">
+    <!-- <ros2_control name="GazeboSimSystem" type="system">
       <hardware>
         <plugin>gz_ros2_control/GazeboSimSystem</plugin>
@@ -236,9 +236,28 @@
     </ros2_control>
     <gazebo>
-      <!-- Joint state publisher -->
       <plugin filename="gz_ros2_control-system" name="gz_ros2_control::GazeboSimROS2ControlPlugin">
           <parameters>$(find eddiebot_description)/config/diff_drive_controller.yaml</parameters>
       </plugin>
-    </gazebo>
+    </gazebo> -->
+    <ros2_control name="RealSystem" type="system">
+      <hardware>
+        <plugin>eddiebot_description/DiffBotSystemHardware</plugin>
+        <param name="left_wheel_name">left_wheel_joint</param>
+        <param name="right_wheel_name">right_wheel_joint</param>
+        <param name="device">/dev/ttyACM0</param>
+        <param name="baud_rate">115200</param>
+        <param name="timeout_ms">1000</param>
+      </hardware>
+      <joint name="left_wheel_joint">
+        <command_interface name="velocity"/>
+        <state_interface name="position"/>
+        <state_interface name="velocity"/>
+      </joint>
+      <joint name="right_wheel_joint">
+        <command_interface name="velocity"/>
+        <state_interface name="position"/>
+        <state_interface name="velocity"/>
+      </joint>
+    </ros2_control>
   </xacro:macro>
 </robot>
