Commit message: Added changes

File: eddiebot_description/urdf/robots/eddiebot.urdf.xacro (robot description, xacro)
@@ -4,7 +4,12 @@
   <xacro:include filename="$(find eddiebot_description)/urdf/stacks/layer1.urdf.xacro"/>
   <xacro:include filename="$(find eddiebot_description)/urdf/stacks/camera_stand.urdf.xacro"/>
+  <xacro:include filename="$(find eddiebot_description)/urdf/sensors/rplidar.urdf.xacro" />
   <!-- eddiebot -->
   <xacro:base/>
   <xacro:layer1 parent="base_link"/>
-  <xacro:camera_stand parent="plate_0_link"/>
+  <!-- <xacro:camera_stand parent="plate_0_link"/> -->
+  <xacro:rplidar name="rplidar" parent_link="plate_0_link">
+    <origin xyz="0 0 0.035"
+            rpy="0 0 ${pi/2}"/>
+  </xacro:rplidar>
 </robot>

File: eddiebot_description/urdf/stacks/base.urdf.xacro (robot description, xacro)
@@ -241,30 +241,4 @@
       </plugin>
     </gazebo>
-    <!-- Diff Drive -->
-    <!-- <gazebo>
-      <plugin filename="gz-sim-diff-drive-system" name="gz::sim::systems::DiffDrive">
-        <left_joint>left_wheel_joint</left_joint>
-        <right_joint>right_wheel_joint</right_joint>
-        <wheel_separation>${wheel_y_offset*2 + battery_box_width}</wheel_separation>
-        <wheel_radius>${wheel_radius}</wheel_radius>
-        <odom_publish_frequency>1</odom_publish_frequency>
-        <topic>cmd_vel</topic>
-        <frame_id>odom</frame_id>
-        <child_frame_id>base_footprint</child_frame_id>
-        <odom_topic>wheel_odom</odom_topic>
-      </plugin>
-      <plugin filename="gz-sim-joint-state-publisher-system" name="gz::sim::systems::JointStatePublisher">
-        <joint_name>left_wheel_joint</joint_name>
-        <joint_name>right_wheel_joint</joint_name>
-        <topic>model/eddiebot/joint_states</topic>
-      </plugin>
-    </gazebo> -->
-    <!-- create two instances of the ultrasonic sensor -->
-    <!-- <xacro:ultrasonic_sensor topic_name="ultrasonic1" sensor_name="usen1" link_name="ul1" joint_name='uj1' parent="base_link" x="0.195" y="0.09" z="0.015" roll="0" pitch="0" yaw="${M_PI/8}"/>
-    <xacro:ultrasonic_sensor topic_name="ultrasonic2" sensor_name="usen2" link_name="ul2" joint_name='uj2' parent="base_link" x="0.195" y="-0.09" z="0.015" roll="0" pitch="0" yaw="${-M_PI/8}"/> -->
-    <!-- create three instances of the infrared sensor -->
-    <!-- <xacro:infrared_sensor topic_name="infrared1" sensor_name="isen1" link_name="il1" joint_name='ij1' parent="base_link" x="0.135" y="-0.155" z="0.025" roll="0" pitch="0" yaw="${-M_PI/4}"/>
-    <xacro:infrared_sensor topic_name="infrared2" sensor_name="isen2" link_name="il2" joint_name='ij2' parent="base_link" x="0.210" y="0.00" z="0.025" roll="0" pitch="0" yaw="0"/>
-    <xacro:infrared_sensor topic_name="infrared3" sensor_name="isen3" link_name="il3" joint_name='ij3' parent="base_link" x="0.135" y="0.155" z="0.025" roll="0" pitch="0" yaw="${M_PI/4}"/> -->
   </xacro:macro>
 </robot>

Commit message: Updated URDF

File: eddiebot_description/urdf/robots/eddiebot.urdf.xacro (robot description, xacro)
@@ -5,4 +5,6 @@
   <xacro:include filename="$(find eddiebot_description)/urdf/stacks/camera_stand.urdf.xacro"/>
   <xacro:include filename="$(find eddiebot_description)/urdf/sensors/rplidar.urdf.xacro" />
+  <xacro:include filename="$(find eddiebot_description)/urdf/utils/l_bracket.urdf.xacro" />
+  <xacro:include filename="$(find eddiebot_description)/urdf/utils/uv_lamp.urdf.xacro" />
   <!-- eddiebot -->
   <xacro:base/>
@@ -10,6 +12,15 @@
   <!-- <xacro:camera_stand parent="plate_0_link"/> -->
   <xacro:rplidar name="rplidar" parent_link="plate_0_link">
-    <origin xyz="0 0 0.035"
-            rpy="0 0 ${pi/2}"/>
+    <origin xyz="0 0 0.05"
+            rpy="0 0 ${pi}"/>
   </xacro:rplidar>
+  <xacro:l_bracket name="left_lamp_holder" parent_link="plate_0_link">
+      <origin xyz="0.1 0.0 0.00475" rpy="0 0 ${-pi/2}"/>
+  </xacro:l_bracket>
+  <xacro:l_bracket name="right_lamp_holder" parent_link="plate_0_link">
+      <origin xyz="-0.1 0.0 0.00475" rpy="0 0 ${-pi/2}"/>
+  </xacro:l_bracket>
+  <xacro:uv_lamp name="uv_lamp" parent_link="left_lamp_holder_link">
+      <origin xyz="-0.045 -0.1 0.19" rpy="${pi/2} 0 ${pi/2}"/>
+  </xacro:uv_lamp>
 </robot>

File: eddiebot_description/urdf/sensors/rplidar.urdf.xacro (robot description, xacro)
@@ -1,18 +1,5 @@
 <?xml version="1.0"?>
 <robot xmlns:xacro="http://ros.org/wiki/xacro">
-<xacro:macro name="inertial_cuboid_with_pose" params="mass x y z *origin">
-  <inertial>
-    <mass value="${mass}" />
-    <xacro:insert_block name="origin"/>
-    <inertia ixx="${(1/12) * mass * (y*y + z*z)}" ixy="0.0" ixz="0.0"
-      iyy="${(1/12) * mass * (x*x + z*z)}" iyz="0.0"
-      izz="${(1/12) * mass * (x*x + y*y)}" />
-  </inertial>
-</xacro:macro>
-<xacro:macro name="inertial_cuboid" params="mass x y z">
-  <xacro:inertial_cuboid_with_pose mass="${mass}" x="${x}" y="${y}" z="${z}">
-    <origin xyz="0 0 0" />
-  </xacro:inertial_cuboid_with_pose>
-</xacro:macro>
+<xacro:include filename="$(find eddiebot_description)/urdf/utils/inertials.urdf.xacro"/>
 <xacro:macro name="rplidar" params="name parent_link *origin">
   <xacro:property name="cm2m"    value="${1/100.0}"/>

Commit message: Updated code

File: eddiebot_description/urdf/robots/eddiebot.urdf.xacro (robot description, xacro)
@@ -22,5 +22,5 @@
   </xacro:l_bracket>
   <xacro:uv_lamp name="uv_lamp" parent_link="left_lamp_holder_link">
-      <origin xyz="-0.045 -0.1 0.19" rpy="${pi/2} 0 ${pi/2}"/>
+      <origin xyz="0.039 -0.1 0.19" rpy="0 0 0"/>
   </xacro:uv_lamp>
 </robot>

File: eddiebot_description/urdf/utils/uv_lamp.urdf.xacro (robot description, xacro)
@@ -1,50 +1,28 @@
-<?xml version="1.0"?>
 <robot xmlns:xacro="http://ros.org/wiki/xacro">
   <xacro:macro name="uv_lamp" params="name parent_link *origin">
     <link name="${name}_link">
-      <!-- Visual: main rectangular body -->
       <visual>
-        <origin xyz="0 0 0.0" rpy="0 0 0"/>
+        <origin xyz="0 0 0" rpy="0 0 0"/>
         <geometry>
-          <box size="0.24 0.06 0.03"/>
+          <mesh filename="package://eddiebot_description/meshes/Lamp2.stl" scale="0.001 0.001 0.001"/>
         </geometry>
-        <material name="uv_color">
-          <color rgba="0.8 0.8 0.8 1"/>
+        <material name="white">
+          <color rgba="1 1 1 1"/>
         </material>
       </visual>
-      <!-- Visual: cylinder at the back -->
-      <visual>
-        <origin xyz="0.0 0.0 0.015" rpy="0 ${pi/2} 0"/>
+      <collision>
+        <origin xyz="0 0 0" rpy="0 0 0"/>
         <geometry>
-          <cylinder length="0.24" radius="0.03"/>
-        </geometry>
-        <material name="uv_color"/>
-      </visual>
-      <!-- Collision geometry -->
-      <collision>
-        <origin xyz="0 0 0.0" rpy="0 0 0"/>
-        <geometry>
-          <box size="0.18 0.06 0.01"/>
+          <mesh filename="package://eddiebot_description/meshes/Lamp2.stl" scale="0.001 0.001 0.001"/>
         </geometry>
       </collision>
-      <collision>
-        <origin xyz="0 0 -0.01" rpy="0 0 0"/>
-        <geometry>
-          <cylinder length="0.02" radius="0.015"/>
-        </geometry>
-      </collision>
-      <!-- Inertial -->
       <inertial>
         <mass value="1.0"/>
-        <origin xyz="0 0 0.03"/>
-        <inertia ixx="0.0005" ixy="0.0" ixz="0.0"
-                 iyy="0.0005" iyz="0.0"
-                 izz="0.0003"/>
+        <origin xyz="-0.020181 -0.000000002 0.000000001"/>
+        <inertia ixx="0.005460" ixy="0.000000000193" ixz="-0.000000000018"
+                iyy="0.000523" iyz="0.000000000069"
+                izz="0.005257"/>
       </inertial>
     </link>
-    <!-- Gazebo visual material -->
-    <gazebo reference="${name}_link">
-      <material>Gazebo/White</material>
-    </gazebo>
     <joint name="${name}_joint" type="fixed">
       <parent link="${parent_link}"/>
@@ -52,4 +30,7 @@
       <xacro:insert_block name="origin"/>
     </joint>
+    <gazebo reference="${name}_link">
+      <material>Gazebo/White</material>
+    </gazebo>
   </xacro:macro>
 </robot>
